File: WeatherWidget Eagle/WeatherWidget.brd (EAGLE design)
At the start: 33 x 53 mm, 16 parts, among them J1 USB_MINI-B_SMT, SW1 SPST_TACT-EVQQ2

Commit message: updated board info
Parts:
- moved U1 14.8 mm to (12.8, 7.24), turned to 270 degrees
- moved J1 14.7 mm to (27.3, 8.00), turned to 0 degrees
- moved 10UF 2.80 mm to (29.2, 13.5)
- moved U$1 2.16 mm to (2.67, 36.4), turned to 90 degrees
- moved POWER 2.03 mm to (16.4, 12.2)
- moved R1 1.80 mm to (10.9, 15.2)
- moved R2 1.57 mm to (24.9, 16.1)
- moved U$2 0.42 mm to (12.3, 3.64)
Routing:
- net GND: track 69.5 -> 13.9 mm, vias 2 -> 5
- net SCL: track 1.17 -> 24.3 mm
- net RXD: track 53.7 -> 31.2 mm, vias 0 -> 1
- net 5V: track 82.7 -> 67.1 mm, vias 1 -> 2
- net SDA: track 3.31 -> 18.4 mm
- net TXD: track 49.9 -> 37.6 mm, vias 0 -> 1
- net IO0: track 39.8 -> 48.2 mm
- net 3.3V: track 49.5 -> 43.2 mm
- net EN: track 26.7 -> 25.2 mm
- net WBTN: track 21.9 -> 22.7 mm
- net N$1: track 10.1 -> 9.50 mm
- added copper zone on layer 16, net GND
Other:
- board text added: "RXD"
- board text added: "TXD"

Commit message: updated esp32 footprint
Parts:
- ESP32: device bitcows-esp32:ESP-WROOM-03 -> bitcows-esp32:ESP-WROOM-03-HOLES
Connections:
- net GND: now also ESP32.GND1, ESP32.GND2, ESP32.GND3, ESP32.GND4; no longer ESP32.GND01, ESP32.GND02, ESP32.GND03
Routing:
- net GND: track 13.9 -> 30.4 mm
