File: WeatherWidget Eagle/WeatherWidget.sch (EAGLE design)
At the start: 13 parts, among them J1 USB_MINI-B_SMT, SW1 SPST_TACT-EVQQ2

Commit message: updated esp32 footprint
Other:
- moved on the sheet: ESP32
Changed lines of the file:
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@@
 <part name="GND2" library="supply1" library_urn="urn:adsk.eagle:library:371" deviceset="GND" device=""/>
 <part name="GND3" library="supply1" library_urn="urn:adsk.eagle:library:371" deviceset="GND" device=""/>
-<part name="128X1" library="128x64oled" library_urn="urn:adsk.eagle:library:5227684" deviceset="128X64OLED" device="" package3d_urn="urn:adsk.eagle:package:5227687/1"/>
+<part name="128X1" library="128x64oled" library_urn="urn:adsk.eagle:library:5227684" deviceset="128X64OLED" device="" package3d_urn="urn:adsk.eagle:package:5227687/2"/>
 <part name="SW1" library="adafruit" library_urn="urn:adsk.eagle:library:420" deviceset="SPST_TACT" device="-EVQQ2" package3d_urn="urn:adsk.eagle:package:6240643/1"/>
 <part name="R4" library="adafruit" library_urn="urn:adsk.eagle:library:420" deviceset="R-US_" device="R0805" package3d_urn="urn:adsk.eagle:package:6240566/1" value="220"/>
